File: lokho2-rpico-purple/lokho2-rpico-purple.kicad_pcb (KiCad board)
At the start: 2 copper layers, 100 x 100 mm, 10 parts, among them J1 GPIOA, J2 GPIOB, J3 GPIOC, SW1 RUN

Commit message: pcb description
Routing:
- added copper zone on B.Cu, net GND
- added copper zone on F.Cu, net GND
Other:
- board text added: "!RUN"
- board text added: "3V3"
- board text added: "ANALOG"
- board text added: "GENERAL PURPOSE IN-OUT"
- board text added: "GND"
- board text added: "GP0"
- board text added: "GP1"
- board text added: "GP10"
- board text added: "GP11"
- board text added: "GP12"
- board text added: "GP13"
- board text added: "GP14"
- board text added: "GP2"
- board text added: "GP26"
- board text added: "GP27"
- board text added: "GP28"
- board text added: "GP29"
- board text added: "GP3"
- board text added: "GP4"
- board text added: "GP5"
- board text added: "GP6"
- board text added: "GP7"
- board text added: "GP8"
- board text added: "GP9"
